Commit message: Update latest with Udacity workspace

File: udacity_bot/urdf/udacity_bot.xacro (robot description, xacro)
@@ -8,8 +8,4 @@
     <child link="chassis" />
   </joint>
-   <!-- Define Blue -->
-   <material name="blue">
-        <color rgba="1.0 0.0 0.0 1"/>
-   </material>
   <link name='chassis'>
     <pose>0 0 0.1 0 0 0</pose>
@@ -30,5 +26,5 @@
     </collision>
     <visual name='chassis_visual'>
-      <origin xyz="0 0 0" rpy=" 0 0 0"/>
+      <origin xyz="0 0 0" rpy="0 0 0"/>
       <geometry>
         <box size=".4 .2 .1"/>
@@ -36,21 +32,11 @@
     </visual>
     <collision name='back_caster_collision'>
-      <origin xyz="-0.15 0 -0.05" rpy=" 0 0 0"/>
+      <origin xyz="-0.15 0 -0.05" rpy="0 0 0"/>
       <geometry>
-        <sphere radius="0.05"/>
+        <sphere radius="0.0499"/>
       </geometry>
-      <surface>
-        <friction>
-          <ode>
-            <mu>0</mu>
-            <mu2>0</mu2>
-            <slip1>1.0</slip1>
-            <slip2>1.0</slip2>
-          </ode>
-        </friction>
-      </surface>
     </collision>
     <visual name='back_caster_visual'>
-      <origin xyz="-0.15 0 -0.05" rpy=" 0 0 0"/>
+      <origin xyz="-0.15 0 -0.05" rpy="0 0 0"/>
       <geometry>
         <sphere radius="0.05"/>
@@ -58,21 +44,11 @@
     </visual>
     <collision name='front_caster_collision'>
-      <origin xyz="0.15 0 -0.05" rpy=" 0 0 0"/>
+      <origin xyz="0.15 0 -0.05" rpy="0 0 0"/>
       <geometry>
-        <sphere radius="0.05"/>
+        <sphere radius="0.0499"/>
       </geometry>
-      <surface>
-        <friction>
-          <ode>
-            <mu>0</mu>
-            <mu2>0</mu2>
-            <slip1>1.0</slip1>
-            <slip2>1.0</slip2>
-          </ode>
-        </friction>
-      </surface>
     </collision>
     <visual name='front_caster_visual'>
-      <origin xyz="0.15 0 -0.05" rpy=" 0 0 0"/>
+      <origin xyz="0.15 0 -0.05" rpy="0 0 0"/>
       <geometry>
         <sphere radius="0.05"/>
@@ -82,6 +58,6 @@
   <link name="left_wheel">
     <inertial>
-      <origin xyz="0 0 0" rpy="0 1.5707 1.5707"/>
-      <mass value="5"/>
+      <mass value="5.0"/>
+      <origin xyz="0.0 0 0" rpy="0 1.5707 1.5707"/>
       <inertia
           ixx="0.1" ixy="0" ixz="0"
@@ -90,23 +66,18 @@
       />
     </inertial>
+    <collision>
+      <origin xyz="0 0 0" rpy="0 1.5707 1.5707"/>
+       <cylinder radius="0.1" length="0.05"/>
+      <geometry>
+       <cylinder radius="0.1" length="0.05"/>
+      </geometry>
+    </collision>
     <visual>
       <origin xyz="0 0 0" rpy="0 1.5707 1.5707"/>
       <geometry>
-        <cylinder radius="0.1" length="0.05"/>
+       <cylinder radius="0.1" length="0.05"/>
       </geometry>
-      <material name="blue"/>
-        <!--
-        <color rgba="1.0 0.0 0.0 1"/>
-        <color rgba="0.75294 0.75294 0.75294 1"/>
-      </material>
-        -->
+      <material name="red"/>
     </visual>
-    <collision>
-      <origin xyz="0 0 0" rpy="0 1.5707 1.5707"/>
-        <cylinder radius="0.1" length="0.05"/>
-      <geometry>
-        <cylinder radius="0.1" length="0.05"/>
-      </geometry>
-    </collision>
     <joint type="continuous" name="left_wheel_hinge">
       <origin xyz="0 0.15 0" rpy="0 0 0"/>
@@ -120,6 +91,6 @@
   <link name="right_wheel">
     <inertial>
-      <origin xyz="0 0 0" rpy="0 1.5707 1.5707"/>
-      <mass value="5"/>
+      <mass value="5.0"/>
+      <origin xyz="0.0 0 0" rpy="0 1.5707 1.5707"/>
       <inertia
           ixx="0.1" ixy="0" ixz="0"
@@ -128,23 +99,18 @@
       />
     </inertial>
+    <collision>
+      <origin xyz="0 0 0" rpy="0 1.5707 1.5707"/>
+       <cylinder radius="0.1" length="0.05"/>
+      <geometry>
+       <cylinder radius="0.1" length="0.05"/>
+      </geometry>
+    </collision>
     <visual>
       <origin xyz="0 0 0" rpy="0 1.5707 1.5707"/>
       <geometry>
-        <cylinder radius="0.1" length="0.05"/>
+       <cylinder radius="0.1" length="0.05"/>
       </geometry>
-      <material name="blue"/>
-      <!--
-      <material name="red">
-        <color rgba="1.0 0.0 0.0 1"/>
-      </material>
-      -->
+      <material name="red"/>
     </visual>
-    <collision>
-      <origin xyz="0 0 0" rpy="0 1.5707 1.5707"/>
-        <cylinder radius="0.1" length="0.05"/>
-      <geometry>
-        <cylinder radius="0.1" length="0.05"/>
-      </geometry>
-    </collision>
   </link>
   <joint type="continuous" name="left_wheel_hinge">
@@ -164,36 +130,4 @@
     <joint_properties damping="1.0" friction="1.0"/>
   </joint>
-<!--
-  <link name="camera">
-    <inertial>
-      <origin xyz="0 0 0" rpy="0 0 0"/>
-      <mass value="0.1"/>
-      <box_inertia m="0.1" x="0.05" y="0.05" z="0.05" />
-      <inertia
-          ixx="1e-6" ixy="0" ixz="0"
-          iyy="1e-6" iyz="0"
-          izz="1e-6"
-      />
-    </inertial>
-    <visual>
-      <origin xyz="0 0 0" rpy="0 0 0"/>
-      <geometry>
-        <box size="0.05 0.05 0.05"/>
-      </geometry>
-    </visual>
-    <collision>
-      <origin xyz="0 0 0" rpy="0 0 0"/>
-      <geometry>
-        <box size="0.05 0.05 0.05"/>
-      </geometry>
-    </collision>
-    <joint type="fixed" name="camera_joint">
-      <axis xyz="0 1 0" />
-      <origin xyz="0.2 0 0" rpy="0 0 0"/>
-      <child link="camera"/>
-      <parent link="chassis"/>
-    </joint>
-  </link>
--->
     <link name="camera">
     <collision>
@@ -208,5 +142,5 @@
         <box size="0.05 0.05 0.05"/>
       </geometry>
-      <material name="green"/>
+      <material name="red"/>
     </visual>
     <inertial>
@@ -240,5 +174,5 @@
         <mesh filename="package://udacity_bot/meshes/hokuyo.dae"/>
       </geometry>
-      <material name="green"/>
+      <material name="red"/>
     </visual>
     <inertial>
